Commit message: Add files via upload

File: urdf/lj_v7080.xacro (robot description, xacro)
@@ -2,4 +2,5 @@
 <robot xmlns:xacro="http://wiki.ros.org/xacro" name="lj_v7080">
   <xacro:include filename="$(find keyence_experimental)/urdf/lj_v7080_macro.xacro"/>
-  <xacro:lj_v7080 prefix=""/>
+  <xacro:arg name="sim_gazebo" value="false"/>
+  <xacro:lj_v7080 prefix="" sim_gazebo="$(arg sim_gazebo)"/>
 </robot>

File: urdf/lj_v7080_macro.xacro (robot description, xacro)
@@ -1,6 +1,13 @@
 <?xml version="1.0"?>
 <robot xmlns:xacro="http://wiki.ros.org/xacro">
-  <xacro:macro name="lj_v7080" params="prefix">
+  <xacro:include filename="$(find keyence_experimental)/urdf/lj_v7080.gazebo.xacro"/>
+  <xacro:macro name="lj_v7080" params="prefix sim_gazebo">
   <xacro:property name="ref_dist_a" value="0.08"/>
+    <link name="base_link"/>
+    <joint name="base_to_frame" type="fixed">
+      <origin xyz="0 0 -0.05" rpy="0 0 0"/>
+      <parent link="base_link"/>
+      <child link="${prefix}lj_v7080_frame"/>
+    </joint>
     <link name="${prefix}lj_v7080_frame">
       <visual>
@@ -26,8 +33,11 @@
     <link name="${prefix}lj_v7080_optical_frame"/>
     <joint name="optical_frame" type="fixed">
-      <origin xyz="0 0 ${ref_dist_a}" rpy="0 0 0"/>
-      <parent link="${prefix}lj_v7080_optical_frame"/>
-      <child link="${prefix}lj_v7080_frame"/>
+      <origin xyz="0 0 ${-ref_dist_a}" rpy="0 0 ${pi/2}"/>
+      <parent link="${prefix}lj_v7080_frame"/>
+      <child link="${prefix}lj_v7080_optical_frame"/>
    </joint>
+   <xacro:if value="$(arg sim_gazebo)">
+      <xacro:gazebo_keyence prefix="${prefix}"/>
+   </xacro:if>
   </xacro:macro>
 </robot>

Commit message: Add files via upload

File: urdf/lj_v7080.xacro (robot description, xacro)
@@ -2,4 +2,5 @@
 <robot xmlns:xacro="http://wiki.ros.org/xacro" name="lj_v7080">
   <xacro:include filename="$(find keyence_experimental)/urdf/lj_v7080_macro.xacro"/>
-  <xacro:lj_v7080 prefix="" sim_gazebo="false"/>
+  <xacro:arg name="sim_gazebo" value="false"/>
+  <xacro:lj_v7080 prefix="" sim_gazebo="$(arg sim_gazebo)"/>
 </robot>

File: urdf/lj_v7080_macro.xacro (robot description, xacro)
@@ -4,4 +4,10 @@
   <xacro:macro name="lj_v7080" params="prefix sim_gazebo">
   <xacro:property name="ref_dist_a" value="0.08"/>
+    <link name="base_link"/>
+    <joint name="base_to_frame" type="fixed">
+      <origin xyz="0 0 -0.05" rpy="0 0 0"/>
+      <parent link="base_link"/>
+      <child link="${prefix}lj_v7080_frame"/>
+    </joint>
     <link name="${prefix}lj_v7080_frame">
       <visual>
@@ -27,5 +33,5 @@
     <link name="${prefix}lj_v7080_optical_frame"/>
     <joint name="optical_frame" type="fixed">
-      <origin xyz="0 0 ${-ref_dist_a}" rpy="0 0 0"/>
+      <origin xyz="0 0 ${-ref_dist_a}" rpy="0 0 ${pi/2}"/>
       <parent link="${prefix}lj_v7080_frame"/>
       <child link="${prefix}lj_v7080_optical_frame"/>
